File: Hardware/IncubPower.sch (EAGLE design)
At the start: 23 parts, among them T1 BT138-V, T2 BT138-V, X1 22-23-2041, X2 MKDSN1,5/2-5,08, X3 MKDSN1,5/2-5,08, X4 22-23-2021, X5 MKDSN1,5/2-5,08

Commit message: Release version
Version for production
- 3 buttons on control board
Parts:
- R1, R8: device rcl:R-EU_0207/2V -> rcl:R-EU_0204/7
- R7: device resistor:R-EU_0309/V -> resistor:R-EU_0204/7
Changed lines of the file:
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@@
 <part name="F1" library="fuse" deviceset="FUSE" device="BLANK_5X20MM"/>
 <part name="OK1" library="optocoupler" deviceset="MOC30*M" device="" technology="20"/>
-<part name="R1" library="rcl" deviceset="R-EU_" device="0207/2V" value="390"/>
+<part name="R1" library="rcl" deviceset="R-EU_" device="0204/7" value="390"/>
 <part name="R2" library="rcl" deviceset="R-EU_" device="R0805" value="330"/>
 <part name="X2" library="con-phoenix-508" deviceset="MKDSN1,5/2-5,08" device=""/>
@@
 <part name="R6" library="rcl" deviceset="R-EU_" device="R0805" value="1 k [NP]"/>
 <part name="GND6" library="supply1" deviceset="GND" device=""/>
-<part name="R7" library="resistor" deviceset="R-EU_" device="0309/V" value="68 k"/>
+<part name="R7" library="resistor" deviceset="R-EU_" device="0204/7" value="68 k"/>
 <part name="X4" library="con-molex" deviceset="22-23-2021" device=""/>
 <part name="OK4" library="optocoupler" deviceset="MOC30*M" device="" technology="20"/>
 <part name="T2" library="triac" deviceset="BT138" device="-V"/>
-<part name="R8" library="rcl" deviceset="R-EU_" device="0207/2V" value="390"/>
+<part name="R8" library="rcl" deviceset="R-EU_" device="0204/7" value="390"/>
 <part name="R9" library="rcl" deviceset="R-EU_" device="R0805" value="330"/>
 <part name="X5" library="con-phoenix-508" deviceset="MKDSN1,5/2-5,08" device=""/>
